File: PCBs/IOExpanderVersion.sch (KiCad schematic (older format))
At the start: 14 parts, among them J1 Conn_01x04_Male, J10 Conn_01x04_Male, J2 Conn_01x05_Male, J3 Conn_01x05_Male, J4 Conn_01x02_Male, J5 Conn_01x02_Male, J6 Conn_01x02_Male, J7 Conn_01x02_Male, J8 Conn_01x03_Male, J9 Conn_01x03_Male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

Commit message: Updated to new kicad 5.x
Parts:
- U1: footprint SMD_Packages:SOIC-28 -> Housings_SOIC:SOIC-28W_7.5x17.9mm_Pitch1.27mm
Changed lines of the file:
@@
 F 0 "U1" H 4800 4475 50  0000 R CNN
 F 1 "MCP23017" H 4800 4400 50  0000 R CNN
-F 2 "SMD_Packages:SOIC-28" H 4950 2500 50  0001 L CNN
+F 2 "Housings_SOIC:SOIC-28W_7.5x17.9mm_Pitch1.27mm" H 4950 2500 50  0001 L CNN
 F 3 "" H 5150 4450 50  0001 C CNN
 	1    4900 3450
